File: Hardware/MyoWare_Proto_Shield.brd (EAGLE design)
At the start: 52.1 x 20.8 mm, 27 parts

Commit message: Removed RoHS compliance claim
Parts:
- removed U$3: (no value), advancer-technologies:ROHS
Changed lines of the file:
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@@
 <?xml version="1.0" encoding="utf-8"?>
 <!DOCTYPE eagle SYSTEM "eagle.dtd">
-<eagle version="7.3.2">
+<eagle version="7.4.0">
 <drawing>
 <settings>
@@
 </autorouter>
 <elements>
-<element name="U$3" library="advancer-technologies" package="ROHS" value="" x="-19.05" y="-8.0645" smashed="yes" rot="MR0"/>
 <element name="JP19" library="SparkFun-Connectors" package="1X03_NO_SILK" value="Power" x="24.5745" y="2.54" smashed="yes" rot="R270"/>
 <element name="U$9" library="advancer-technologies" package="SPIRAL_LOGO_60%" value="" x="21.3995" y="6.477"/>
